File: Hardware/PCB/FitnessMotionDevice.kicad_pcb (KiCad board)
At the start: 2 copper layers, 42 x 42 mm, 52 parts, among them J1 USB_C_Receptacle_USB2.0_16P, J2 Conn_01x02_MountingPin, J3 Conn_01x04, J4 Conn_01x04, U1 nRF52840, U2 BQ24074RGT, U3 USBLC6-2SC6, U7 LSM6DSVTR, Y2 Crystal_GND23

Commit message: added readme
Parts:
- added +3V3: TestPoint_Pad_D1.0mm, TestPoint:TestPoint_Pad_D1.0mm, F.Cu at (124.5, 87.2)
- added +5V: TestPoint_Pad_D1.0mm, TestPoint:TestPoint_Pad_D1.0mm, F.Cu at (141.0, 110.5)
- added C26: 100nF, Capacitor_SMD:C_0603_1608Metric, F.Cu at (142.8, 97.2)
- added GND: TestPoint_Pad_D1.0mm, TestPoint:TestPoint_Pad_D1.0mm, F.Cu at (146.8, 110.5)
- added R13: 1M, Resistor_SMD:R_0402_1005Metric, F.Cu at (142.3, 96.0)
- added R4: 1M, Resistor_SMD:R_0402_1005Metric, F.Cu at (142.2, 95.0)
- added VBAT: TestPoint_Pad_D1.0mm, TestPoint:TestPoint_Pad_D1.0mm, F.Cu at (146.8, 108.5)
Connections:
- U1 pad R24: unconnected-(U1-P1.06-PadR24) -> Net-(U1-P1.06)
Routing:
- net /VBAT: track 43.6 -> 60.6 mm, vias 2 -> 4
- net +5V: track 66.6 -> 77.4 mm
- net +3V3: track 134.0 -> 141.1 mm
- net Net-(U1-P1.06): track 0.00 -> 4.64 mm
- net GND: track 89.6 -> 93.0 mm
- net /SWDIO: track 12.6 -> 13.8 mm
Other:
- board text added: "+3V3"
- board text added: "GND"
- board text added: "SCL"
- board text added: "SDA"
- board text added: "SWD"
